File: Circuit/DiffPanTilt.kicad_sch (KiCad schematic)
At the start: 18 parts, among them J1 Power, J2 Stepper 1, J3 Stepper 2, J4 BT, J5 Stepper 1 Power, J6 Stepper 2 Power, J7 12V Input, J8 5V Output, J9 Display, SW1 Switch

Commit message: [Circuit] Change the footprint of J1 to pin socket, and fine tune the PCB layout
Parts:
- J1: footprint Connector_PinHeader_2.54mm:PinHeader_1x04_P2.54mm_Vertical -> Connector_PinSocket_2.54mm:PinSocket_1x04_P2.54mm_Vertical
Changed lines of the file:
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@@
 			)
 		)
-		(property "Footprint" "Connector_PinHeader_2.54mm:PinHeader_1x04_P2.54mm_Vertical"
+		(property "Footprint" "Connector_PinSocket_2.54mm:PinSocket_1x04_P2.54mm_Vertical"
 			(at 55.88 60.96 0)
 			(effects
